File: hardware/ac_onoff_controller/ac_onoff_controller.kicad_pcb (KiCad board)
At the start: 2 copper layers, 100 x 52.5 mm, 40 parts, among them J1 Conn_02x04_Odd_Even, J2 Conn_01x02, M1 Motor_Servo, M2 Motor_Servo, Q1 2SK4017, Q2 2SK4017, Q3 2SC1815, Q6 2SK4017, SW1 SW_SPST, SW2 SW_Push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

Commit message: export gerbers for jlcpcb
Parts:
- added D7: D, Diode_THT:D_DO-15_P12.70mm_Horizontal, F.Cu at (75.4, 74.7)
- D1: moved to F.Cu
- RV1: value R_Potentiometer_Trim -> 20k
Routing:
- net Net-(D7-K): track 11.0 -> 27.2 mm
- net VCC: track 203.1 -> 208.0 mm
- net GND: track 281.2 -> 281.9 mm, vias 111 -> 113
