File: hardware/ac_onoff_controller/ac_onoff_controller.kicad_sch (KiCad schematic)
At the start: 41 parts, among them J1 Conn_02x04_Odd_Even, J2 Conn_01x02, M1 Motor_Servo, M2 Motor_Servo, Q1 2SK4017, Q2 2SK4017, Q3 2SC1815, Q6 2SK4017, SW1 SW_SPST, SW2 SW_Push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

Commit message: add the MPN of DHT20
Parts:
- D7, H1, H2, H3, H4: purchase (none) -> 0
- U2: MPN (none) -> DHT20; URL (none) -> https://akizukidenshi.com/catalog/g/g116732/; purchase (none) -> 1
Changed lines of the file:
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@@
+      (effects (font (size 1.27 1.27)) hide)
+    )
+    (property "purchase" "0" (at 67.31 185.42 0)
       (effects (font (size 1.27 1.27)) hide)
     )
@@
       (effects (font (size 1.27 1.27)) hide)
     )
+    (property "MPN" "DHT20" (at 74.93 138.43 0)
+      (effects (font (size 1.27 1.27)) hide)
+    )
+    (property "URL" "https://akizukidenshi.com/catalog/g/g116732/" (at 74.93 138.43 0)
+      (effects (font (size 1.27 1.27)) hide)
+    )
+    (property "purchase" "1" (at 74.93 138.43 0)
+      (effects (font (size 1.27 1.27)) hide)
+    )
     (pin "1")
     (pin "2")
@@
       (effects (font (size 1.27 1.27)) hide)
     )
+    (property "purchase" "0" (at 67.31 190.5 0)
+      (effects (font (size 1.27 1.27)) hide)
+    )
     (instances
       (project "ac_onoff_controller"
@@
       (effects (font (size 1.27 1.27)) hide)
     )
+    (property "purchase" "0" (at 67.31 175.26 0)
+      (effects (font (size 1.27 1.27)) hide)
+    )
     (instances
       (project "ac_onoff_controller"
@@
     )
     (property "Sim.Pins" "1=K 2=A" (at 88.9 53.34 0)
+      (effects (font (size 1.27 1.27)) hide)
+    )
+    (property "purchase" "0" (at 88.9 53.34 0)
       (effects (font (size 1.27 1.27)) hide)
     )
@@
       (effects (font (size 1.27 1.27)) hide)
     )
+    (property "purchase" "0" (at 67.31 180.34 0)
+      (effects (font (size 1.27 1.27)) hide)
+    )
